File: ENYA-SIMR-GTWL-PCEN.kicad_pcb (KiCad board)
At the start: 2 copper layers, 22.8 x 25.1 mm, 11 parts, among them J1 PICO_BLADE_1x6_MALE_RA_SMD, SW1 PEC11H-4015F-S0016

Commit message: correction button matrix diode polarity
Parts:
- turned D1 to 0 degrees
Connections:
- D1 pad 1: /BTN_ROW -> Net-(D1-K)
- D1 pad 2: Net-(D1-A) -> /BTN_ROW
- SW1 pad S1: Net-(D1-A) -> Net-(D1-K)
Routing:
- net Net-(D1-K): track 0.00 -> 1.81 mm
- net Net-(D1-A): track 1.81 -> 0.00 mm
Changed lines of the file:
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@@
   (net 3 "/ENC_B")
   (net 4 "/BTN_ROW")
-  (net 5 "Net-(D1-A)")
+  (net 5 "Net-(D1-K)")
   (net 6 "+3.3V")
   (net 7 "/BTN_COL")
@@
       (net 2 "GND") (pinfunction "C") (pintype "passive"))
     (pad "S1" thru_hole circle locked (at -2.5 -7 90) (size 1.524 1.524) (drill 1) (layers "*.Cu" "*.Mask")
-      (net 5 "Net-(D1-A)") (pinfunction "S1") (pintype "passive"))
+      (net 5 "Net-(D1-K)") (pinfunction "S1") (pintype "passive"))
     (pad "S2" thru_hole circle locked (at 2.5 -7 90) (size 1.524 1.524) (drill 1) (layers "*.Cu" "*.Mask")
       (net 7 "/BTN_COL") (pinfunction "S2") (pintype "passive"))
@@
   )
   (footprint "Diode_SMD:D_SOD-123" (layer "B.Cu")
-    (at 213.995 125.603 180)
+    (at 213.995 125.603)
     (descr "SOD-123")
     (tags "SOD-123")
@@
     (fp_line (start 1.4 0.9) (end 1.4 -0.9)
       (stroke (width 0.1) (type solid)) (layer "B.Fab"))
-    (pad "1" smd roundrect (at -1.65 0 180) (size 0.9 1.2) (layers "B.Cu" "B.Paste" "B.Mask") (roundrect_rratio 0.25)
-      (net 4 "/BTN_ROW") (pinfunction "K") (pintype "passive"))
-    (pad "2" smd roundrect (at 1.65 0 180) (size 0.9 1.2) (layers "B.Cu" "B.Paste" "B.Mask") (roundrect_rratio 0.25)
-      (net 5 "Net-(D1-A)") (pinfunction "A") (pintype "passive"))
+    (pad "1" smd roundrect (at -1.65 0) (size 0.9 1.2) (layers "B.Cu" "B.Paste" "B.Mask") (roundrect_rratio 0.25)
+      (net 5 "Net-(D1-K)") (pinfunction "K") (pintype "passive"))
+    (pad "2" smd roundrect (at 1.65 0) (size 0.9 1.2) (layers "B.Cu" "B.Paste" "B.Mask") (roundrect_rratio 0.25)
+      (net 4 "/BTN_ROW") (pinfunction "A") (pintype "passive"))
     (model "${KICAD6_3DMODEL_DIR}/Diode_SMD.3dshapes/D_SOD-123.wrl"
       (offset (xyz 0 0 0))
