File: ENYA-SIMR-GTWL-PCEN.kicad_pcb (KiCad board)
At the start: 2 copper layers, 22.8 x 25.1 mm, 11 parts, among them J1 PICO_BLADE_1x6_MALE_RA_SMD, SW1 PEC11H-4015F-S0016

Commit message: WIP
Parts:
- moved G1 1.66 mm to (213.5, 120.7)
- moved G2 1.28 mm to (214.2, 122.9)
- turned SW1 to 75 degrees
Connections:
- J1 pad 1: +3.3V -> GND
- J1 pad 2: /BTN_COL -> /ENC_B
- J1 pad 3: /BTN_ROW -> /ENC_A
- J1 pad 4: /ENC_A -> /BTN_ROW
- J1 pad 5: /ENC_B -> /BTN_COL
- J1 pad 6: GND -> +3.3V
Routing:
- net /ENC_A: track 14.8 -> 5.94 mm, vias 2 -> 0
- net /ENC_B: track 20.9 -> 13.0 mm
- net /BTN_COL: track 20.2 -> 23.6 mm
- net Net-(D1-K): track 1.81 -> 3.68 mm
- net +3.3V: track 18.5 -> 16.9 mm
- net GND: track 0.00 -> 1.39 mm, vias 28 -> 31
- net Net-(R1-Pad2): track 4.48 -> 5.55 mm
